File: V1/eumesmo-rl-8ch12a-v1.kicad_sch (KiCad schematic)
At the start: 47 parts, among them J1 250-202, J2 250-204, J3 250-204, J4 DB142V-5.08-4P, J5 DB142V-5.08-4P, J6 DB142V-5.08-4P, J7 DB142V-5.08-4P, K1 G5PZ-1A, K2 G5PZ-1A, K3 G5PZ-1A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

Commit message: Adjusted version numbers.
Other:
- title: 8x 24V 12A Relay Module -> eumesmo 8x 24V 12A NO Relay Module
Changed lines of the file:
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@@
 	(paper "A4")
 	(title_block
-		(title "8x 24V 12A Relay Module")
-		(date "2026-06-12")
-		(rev "V1.1")
+		(title "eumesmo 8x 24V 12A NO Relay Module")
+		(date "2026-06-13")
+		(rev "V1.2")
 	)
 	(junction
@@
 		)
 		(instances
-			(project "relay-24v-8ch-12a-v1"
+			(project "eumesmo-rl-8ch12a-v1"
 				(path "/57cfb5e7-a9ab-4784-80b3-e51e693f5cc8"
 					(reference "D13")
@@
 		)
 		(instances
-			(project "relay-24v-8ch-12a-v1"
+			(project "eumesmo-rl-8ch12a-v1"
 				(path "/57cfb5e7-a9ab-4784-80b3-e51e693f5cc8"
 					(reference "#PWR03")
@@
 		)
 		(instances
-			(project "relay-24v-8ch-12a-v1"
+			(project "eumesmo-rl-8ch12a-v1"
 				(path "/57cfb5e7-a9ab-4784-80b3-e51e693f5cc8"
 					(reference "RV5")
@@
 		)
 		(instances
-			(project "relay-24v-8ch-12a-v1"
+			(project "eumesmo-rl-8ch12a-v1"
 				(path "/57cfb5e7-a9ab-4784-80b3-e51e693f5cc8"
 					(reference "J4")
@@
 		)
 		(instances
-			(project "relay-24v-8ch-12a-v1"
+			(project "eumesmo-rl-8ch12a-v1"
 				(path "/57cfb5e7-a9ab-4784-80b3-e51e693f5cc8"
 					(reference "J5")
@@
 		)
 		(instances
-			(project "relay-24v-8ch-12a-v1"
+			(project "eumesmo-rl-8ch12a-v1"
 				(path "/57cfb5e7-a9ab-4784-80b3-e51e693f5cc8"
 					(reference "D7")
@@
 		)
 		(instances
-			(project "relay-24v-8ch-12a-v1"
+			(project "eumesmo-rl-8ch12a-v1"
 				(path "/57cfb5e7-a9ab-4784-80b3-e51e693f5cc8"
 					(reference "K7")
@@
 		)
 		(instances
-			(project "relay-24v-8ch-12a-v1"
+			(project "eumesmo-rl-8ch12a-v1"
 				(path "/57cfb5e7-a9ab-4784-80b3-e51e693f5cc8"
 					(reference "K3")
@@
 		)
 		(instances
-			(project "relay-24v-8ch-12a-v1"
+			(project "eumesmo-rl-8ch12a-v1"
 				(path "/57cfb5e7-a9ab-4784-80b3-e51e693f5cc8"
 					(reference "R6")
@@
 		)
 		(instances
-			(project "relay-24v-8ch-12a-v1"
+			(project "eumesmo-rl-8ch12a-v1"
 				(path "/57cfb5e7-a9ab-4784-80b3-e51e693f5cc8"
 					(reference "D2")
@@
 		)
 		(instances
-			(project "relay-24v-8ch-12a-v1"
+			(project "eumesmo-rl-8ch12a-v1"
 				(path "/57cfb5e7-a9ab-4784-80b3-e51e693f5cc8"
 					(reference "#PWR010")
@@
 		)
 		(instances
-			(project "relay-24v-8ch-12a-v1"
+			(project "eumesmo-rl-8ch12a-v1"
 				(path "/57cfb5e7-a9ab-4784-80b3-e51e693f5cc8"
 					(reference "D12")
@@
 		)
 		(instances
-			(project "relay-24v-8ch-12a-v1"
+			(project "eumesmo-rl-8ch12a-v1"
 				(path "/57cfb5e7-a9ab-4784-80b3-e51e693f5cc8"
 					(reference "R8")
@@
 		)
 		(instances
-			(project "relay-24v-8ch-12a-v1"
+			(project "eumesmo-rl-8ch12a-v1"
 				(path "/57cfb5e7-a9ab-4784-80b3-e51e693f5cc8"
 					(reference "#PWR07")
@@
 		)
 		(instances
-			(project "relay-24v-8ch-12a-v1"
+			(project "eumesmo-rl-8ch12a-v1"
 				(path "/57cfb5e7-a9ab-4784-80b3-e51e693f5cc8"
 					(reference "J6")
@@
 		)
 		(instances
-			(project "relay-24v-8ch-12a-v1"
+			(project "eumesmo-rl-8ch12a-v1"
 				(path "/57cfb5e7-a9ab-4784-80b3-e51e693f5cc8"
 					(reference "D9")
@@
 		)
 		(instances
-			(project "relay-24v-8ch-12a-v1"
+			(project "eumesmo-rl-8ch12a-v1"
 				(path "/57cfb5e7-a9ab-4784-80b3-e51e693f5cc8"
 					(reference "R1")
@@
 		)
 		(instances
-			(project "relay-24v-8ch-12a-v1"
+			(project "eumesmo-rl-8ch12a-v1"
 				(path "/57cfb5e7-a9ab-4784-80b3-e51e693f5cc8"
 					(reference "J2")
@@
 		)
 		(instances
-			(project "relay-24v-8ch-12a-v1"
+			(project "eumesmo-rl-8ch12a-v1"
 				(path "/57cfb5e7-a9ab-4784-80b3-e51e693f5cc8"
 					(reference "#PWR04")
@@
 		)
 		(instances
-			(project "relay-24v-8ch-12a-v1"
+			(project "eumesmo-rl-8ch12a-v1"
 				(path "/57cfb5e7-a9ab-4784-80b3-e51e693f5cc8"
 					(reference "R5")
@@
 		)
 		(instances
-			(project "relay-24v-8ch-12a-v1"
+			(project "eumesmo-rl-8ch12a-v1"
 				(path "/57cfb5e7-a9ab-4784-80b3-e51e693f5cc8"
 					(reference "D5")
@@
 		)
 		(instances
-			(project "relay-24v-8ch-12a-v1"
+			(project "eumesmo-rl-8ch12a-v1"
 				(path "/57cfb5e7-a9ab-4784-80b3-e51e693f5cc8"
 					(reference "#FLG01")
@@
 		)
 		(instances
-			(project "relay-24v-8ch-12a-v1"
+			(project "eumesmo-rl-8ch12a-v1"
 				(path "/57cfb5e7-a9ab-4784-80b3-e51e693f5cc8"
 					(reference "R3")
@@
 		)
 		(instances
-			(project "relay-24v-8ch-12a-v1"
+			(project "eumesmo-rl-8ch12a-v1"
 				(path "/57cfb5e7-a9ab-4784-80b3-e51e693f5cc8"
 					(reference "K4")
@@
 		)
 		(instances
-			(project "relay-24v-8ch-12a-v1"
+			(project "eumesmo-rl-8ch12a-v1"
 				(path "/57cfb5e7-a9ab-4784-80b3-e51e693f5cc8"
 					(reference "D15")
@@
 		)
 		(instances
-			(project "relay-24v-8ch-12a-v1"
+			(project "eumesmo-rl-8ch12a-v1"
 				(path "/57cfb5e7-a9ab-4784-80b3-e51e693f5cc8"
 					(reference "RV8")
@@
 		)
 		(instances
-			(project "relay-24v-8ch-12a-v1"
+			(project "eumesmo-rl-8ch12a-v1"
 				(path "/57cfb5e7-a9ab-4784-80b3-e51e693f5cc8"
 					(reference "J7")
@@
 		)
 		(instances
-			(project "relay-24v-8ch-12a-v1"
+			(project "eumesmo-rl-8ch12a-v1"
 				(path "/57cfb5e7-a9ab-4784-80b3-e51e693f5cc8"
 					(reference "J3")
@@
 		)
 		(instances
-			(project "relay-24v-8ch-12a-v1"
+			(project "eumesmo-rl-8ch12a-v1"
 				(path "/57cfb5e7-a9ab-4784-80b3-e51e693f5cc8"
 					(reference "K5")
@@
 		)
 		(instances
-			(project "relay-24v-8ch-12a-v1"
+			(project "eumesmo-rl-8ch12a-v1"
 				(path "/57cfb5e7-a9ab-4784-80b3-e51e693f5cc8"
 					(reference "K1")
@@
 		)
 		(instances
-			(project "relay-24v-8ch-12a-v1"
+			(project "eumesmo-rl-8ch12a-v1"
 				(path "/57cfb5e7-a9ab-4784-80b3-e51e693f5cc8"
 					(reference "D16")
@@
 		)
 		(instances
-			(project "relay-24v-8ch-12a-v1"
+			(project "eumesmo-rl-8ch12a-v1"
 				(path "/57cfb5e7-a9ab-4784-80b3-e51e693f5cc8"
 					(reference "#PWR06")
@@
 		)
 		(instances
-			(project "relay-24v-8ch-12a-v1"
+			(project "eumesmo-rl-8ch12a-v1"
 				(path "/57cfb5e7-a9ab-4784-80b3-e51e693f5cc8"
 					(reference "RV4")
@@
 		)
 		(instances
-			(project "relay-24v-8ch-12a-v1"
+			(project "eumesmo-rl-8ch12a-v1"
 				(path "/57cfb5e7-a9ab-4784-80b3-e51e693f5cc8"
 					(reference "R4")
@@
 		)
 		(instances
-			(project "relay-24v-8ch-12a-v1"
+			(project "eumesmo-rl-8ch12a-v1"
 				(path "/57cfb5e7-a9ab-4784-80b3-e51e693f5cc8"
 					(reference "D1")
@@
 		)
 		(instances
-			(project "relay-24v-8ch-12a-v1"
+			(project "eumesmo-rl-8ch12a-v1"
 				(path "/57cfb5e7-a9ab-4784-80b3-e51e693f5cc8"
 					(reference "RV2")
@@
 		)
 		(instances
-			(project "relay-24v-8ch-12a-v1"
+			(project "eumesmo-rl-8ch12a-v1"
 				(path "/57cfb5e7-a9ab-4784-80b3-e51e693f5cc8"
 					(reference "J1")
@@
 		)
 		(instances
-			(project "relay-24v-8ch-12a-v1"
+			(project "eumesmo-rl-8ch12a-v1"
 				(path "/57cfb5e7-a9ab-4784-80b3-e51e693f5cc8"
 					(reference "R7")
@@
 		)
 		(instances
-			(project "relay-24v-8ch-12a-v1"
+			(project "eumesmo-rl-8ch12a-v1"
 				(path "/57cfb5e7-a9ab-4784-80b3-e51e693f5cc8"
 					(reference "R2")
@@
 		)
 		(instances
-			(project "relay-24v-8ch-12a-v1"
+			(project "eumesmo-rl-8ch12a-v1"
 				(path "/57cfb5e7-a9ab-4784-80b3-e51e693f5cc8"
 					(reference "#PWR05")
@@
 		)
 		(instances
-			(project "relay-24v-8ch-12a-v1"
+			(project "eumesmo-rl-8ch12a-v1"
 				(path "/57cfb5e7-a9ab-4784-80b3-e51e693f5cc8"
 					(reference "#PWR08")
@@
 		)
 		(instances
-			(project "relay-24v-8ch-12a-v1"
+			(project "eumesmo-rl-8ch12a-v1"
 				(path "/57cfb5e7-a9ab-4784-80b3-e51e693f5cc8"
 					(reference "D11")
@@
 		)
 		(instances
-			(project "relay-24v-8ch-12a-v1"
+			(project "eumesmo-rl-8ch12a-v1"
 				(path "/57cfb5e7-a9ab-4784-80b3-e51e693f5cc8"
 					(reference "RV7")
@@
 		)
 		(instances
-			(project "relay-24v-8ch-12a-v1"
+			(project "eumesmo-rl-8ch12a-v1"
 				(path "/57cfb5e7-a9ab-4784-80b3-e51e693f5cc8"
 					(reference "D14")
@@
 		)
 		(instances
-			(project "relay-24v-8ch-12a-v1"
+			(project "eumesmo-rl-8ch12a-v1"
 				(path "/57cfb5e7-a9ab-4784-80b3-e51e693f5cc8"
 					(reference "D8")
@@
 		)
 		(instances
-			(project "relay-24v-8ch-12a-v1"
+			(project "eumesmo-rl-8ch12a-v1"
 				(path "/57cfb5e7-a9ab-4784-80b3-e51e693f5cc8"
 					(reference "K8")
@@
 		)
 		(instances
-			(project "relay-24v-8ch-12a-v1"
+			(project "eumesmo-rl-8ch12a-v1"
 				(path "/57cfb5e7-a9ab-4784-80b3-e51e693f5cc8"
 					(reference "RV6")
@@
 		)
 		(instances
-			(project "relay-24v-8ch-12a-v1"
+			(project "eumesmo-rl-8ch12a-v1"
 				(path "/57cfb5e7-a9ab-4784-80b3-e51e693f5cc8"
 					(reference "#PWR09")
@@
 		)
 		(instances
-			(project "relay-24v-8ch-12a-v1"
+			(project "eumesmo-rl-8ch12a-v1"
 				(path "/57cfb5e7-a9ab-4784-80b3-e51e693f5cc8"
 					(reference "D6")
@@
 		)
 		(instances
-			(project "relay-24v-8ch-12a-v1"
+			(project "eumesmo-rl-8ch12a-v1"
 				(path "/57cfb5e7-a9ab-4784-80b3-e51e693f5cc8"
 					(reference "D3")
@@
 		)
 		(instances
-			(project "relay-24v-8ch-12a-v1"
+			(project "eumesmo-rl-8ch12a-v1"
 				(path "/57cfb5e7-a9ab-4784-80b3-e51e693f5cc8"
 					(reference "D4")
@@
 		)
 		(instances
-			(project "relay-24v-8ch-12a-v1"
+			(project "eumesmo-rl-8ch12a-v1"
 				(path "/57cfb5e7-a9ab-4784-80b3-e51e693f5cc8"
 					(reference "K6")
@@
 		)
 		(instances
-			(project "relay-24v-8ch-12a-v1"
+			(project "eumesmo-rl-8ch12a-v1"
 				(path "/57cfb5e7-a9ab-4784-80b3-e51e693f5cc8"
 					(reference "RV1")
@@
 		)
 		(instances
-			(project "relay-24v-8ch-12a-v1"
+			(project "eumesmo-rl-8ch12a-v1"
 				(path "/57cfb5e7-a9ab-4784-80b3-e51e693f5cc8"
 					(reference "#PWR01")
@@
 		)
 		(instances
-			(project "relay-24v-8ch-12a-v1"
+			(project "eumesmo-rl-8ch12a-v1"
 				(path "/57cfb5e7-a9ab-4784-80b3-e51e693f5cc8"
 					(reference "RV3")
@@
 		)
 		(instances
-			(project "relay-24v-8ch-12a-v1"
+			(project "eumesmo-rl-8ch12a-v1"
 				(path "/57cfb5e7-a9ab-4784-80b3-e51e693f5cc8"
 					(reference "K2")
@@
 		)
 		(instances
-			(project "relay-24v-8ch-12a-v1"
+			(project "eumesmo-rl-8ch12a-v1"
 				(path "/57cfb5e7-a9ab-4784-80b3-e51e693f5cc8"
 					(reference "D10")
